Commit message: weights

File: src/edna_description/urdf/parts/back_leg.xacro (robot description, xacro)
@@ -10,5 +10,5 @@
     <xacro:macro name = "back_leg" params = "prefix parent *origin">
         <link name = "${prefix}_back_leg_link">
-            <xacro:inertial_box mass = "1" x = "${back_leg_length}" y = "${back_leg_width}" z = "${back_leg_height}">
+            <xacro:inertial_box mass = "2.494758035" x = "${back_leg_length}" y = "${back_leg_width}" z = "${back_leg_height}">
                 <origin xyz = "0 0 ${back_leg_height/2}" rpy = "0 0 0"/>
             </xacro:inertial_box>

File: src/edna_description/urdf/parts/elevator.xacro (robot description, xacro)
@@ -14,5 +14,5 @@
     <xacro:macro name = "elevator" params = "prefix parent *origin">
         <link name = "${prefix}_outer_1_link">
-            <xacro:inertial_box mass = "1" x = "${elevator_outer_length}" y = "${elevator_outer_width}" z = "${elevator_outer_height}">
+            <xacro:inertial_box mass = "0.90718474" x = "${elevator_outer_length}" y = "${elevator_outer_width}" z = "${elevator_outer_height}">
                 <origin xyz = "0 0 ${elevator_outer_height/2}" rpy = "0 0 0"/>
             </xacro:inertial_box>
@@ -54,5 +54,5 @@
         </joint>
         <link name = "${prefix}_center_link">
-            <xacro:inertial_box mass = "1" x = "${elevator_outer_length}" y = "${elevator_outer_width}" z = "${elevator_outer_height}">
+            <xacro:inertial_box mass = "1.220163475" x = "${elevator_outer_length}" y = "${elevator_outer_width}" z = "${elevator_outer_height}">
                 <origin xyz = "0 0 ${elevator_outer_height/2}" rpy = "0 0 0"/>
             </xacro:inertial_box>
@@ -94,5 +94,5 @@
         </joint>
         <link name = "${prefix}_outer_2_link">
-            <xacro:inertial_box mass = "1" x = "${elevator_outer_length}" y = "${elevator_outer_width}" z = "${elevator_outer_height}">
+            <xacro:inertial_box mass = "0.90718474" x = "${elevator_outer_length}" y = "${elevator_outer_width}" z = "${elevator_outer_height}">
                 <origin xyz = "0 0 ${elevator_outer_height/2}" rpy = "0 0 0"/>
             </xacro:inertial_box>

File: src/edna_description/urdf/parts/elevator_leg.xacro (robot description, xacro)
@@ -11,5 +11,5 @@
     <xacro:macro name = "elevator_leg" params = "prefix parent *origin">
         <link name = "${prefix}_elevator_leg_link">
-            <xacro:inertial_box mass = "1" x = "${elevator_leg_length}" y = "${elevator_leg_width}" z = "${elevator_leg_height}">
+            <xacro:inertial_box mass = "2.948350405" x = "${elevator_leg_length}" y = "${elevator_leg_width}" z = "${elevator_leg_height}">
                 <origin xyz = "0 0 ${elevator_leg_height/2}" rpy = "0 0 0"/>
             </xacro:inertial_box>
@@ -34,5 +34,5 @@
         </joint>
         <link name = "${prefix}_roller_bar_link">
-            <xacro:inertial_box mass = "1" x = "${roller_bar_length}" y = "${roller_bar_width}" z = "${roller_bar_height}">
+            <xacro:inertial_box mass = "1.093157612" x = "${roller_bar_length}" y = "${roller_bar_width}" z = "${roller_bar_height}">
                 <origin xyz = "0 0 ${roller_bar_height/2}" rpy = "${pi/2} 0 0"/>
             </xacro:inertial_box>

File: src/edna_description/urdf/parts/gripper.xacro (robot description, xacro)
@@ -15,4 +15,7 @@
     <!-- BAR -->
     <link name="${prefix}_gripper_bar_link">
+      <xacro:inertial_box mass = "${1.587573295/3}" x = "${gripper_bar_length}" y = "${gripper_bar_width}" z = "${gripper_bar_height}">
+        <origin xyz = "0 0 0" rpy = "0 0 0"/>
+      </xacro:inertial_box>
       <visual>
         <origin xyz="0 0 0" rpy="0 0 0"/>
@@ -36,4 +39,7 @@
     <!-- Left -->
     <link name="${prefix}_gripper_left_arm_link">
+      <xacro:inertial_box mass = "${1.587573295/3}" x = "${gripper_ar_length}" y = "${gripper_ar_width}" z = "${gripper_ar_height}">
+        <origin xyz = "0 0 0" rpy = "0 0 0"/>
+      </xacro:inertial_box>
       <visual>
         <!-- Alignment Values -->
@@ -66,4 +72,7 @@
     <!-- Right -->
     <link name="${prefix}_gripper_right_arm_link">
+      <xacro:inertial_box mass = "${1.587573295/3}" x = "${gripper_ar_length}" y = "${gripper_ar_width}" z = "${gripper_ar_height}">
+        <origin xyz = "0 0 0" rpy = "0 0 0"/>
+      </xacro:inertial_box>
       <visual>
         <!-- Alignment Values -->

File: src/edna_description/urdf/parts/slider.xacro (robot description, xacro)
@@ -6,5 +6,5 @@
   <xacro:macro name="slider" params="prefix parent *origin">
     <link name = "${prefix}_slider_link">
-        <xacro:inertial_box mass = "1" x = "${slider_block_length}" y = "${slider_block_width}" z = "${slider_block_height}">
+        <xacro:inertial_box mass = "0.90718474" x = "${slider_block_length}" y = "${slider_block_width}" z = "${slider_block_height}">
             <origin xyz = "0 0 0" rpy = "0 0 0"/>
         </xacro:inertial_box>

File: src/edna_description/urdf/parts/square_chassis.xacro (robot description, xacro)
@@ -5,5 +5,5 @@
   <xacro:property name="chassis_width" value=".7366" />
   <xacro:property name="chassis_height" value="0.05588" />
-  <xacro:property name="chassis_weight" value="19.0508795" />
+  <xacro:property name="chassis_weight" value="38.55535145" />
   <xacro:macro name="square_chassis" params="prefix parent *origin">
     <link name="${prefix}_chassis_link">

File: src/edna_description/urdf/parts/zed_macro.urdf.xacro (robot description, xacro)
@@ -62,4 +62,7 @@
     <!-- Camera Center -->
     <link name="${prefix}_camera_center">
+      <xacro:inertial_box mass="0.23" x="0.17525" y="0.03025" z="0.0431">
+        <origin xyz="${screw_offset_x} 0 0 0 0" rpy="0 0 0" />
+      </xacro:inertial_box>
       <visual>
         <origin xyz="${screw_offset_x} 0 0" rpy="0 0 0"/>

File: src/edna_description/urdf/robots/edna.urdf.xacro (robot description, xacro)
@@ -69,9 +69,4 @@
     <origin xyz = "${slider_pos}" rpy = "0 0 0" />
   </xacro:slider>
-  <!-- Bottom Intake + Gripper -->
-  <xacro:property name= "intake_pos" value = "0 0 -${elevator_leg_height/4 + 0.01}" />
-  <xacro:intake prefix="bottom" parent="arm_elevator_leg_link">
-    <origin xyz = "${intake_pos}" rpy = "0 -${pi/2 - 0.05} 0" />
-  </xacro:intake>
   <!-- Control -->
   <xacro:swerve_drive_control plugin="$(arg hw_interface_plugin)"/>
