Commit message: map

File: src/edna_description/urdf/parts/gripper.xacro (robot description, xacro)
@@ -39,5 +39,5 @@
     <!-- Left -->
     <link name="${prefix}_gripper_left_arm_link">
-      <xacro:inertial_box mass = "${1.587573295/3}" x = "${gripper_ar_length}" y = "${gripper_ar_width}" z = "${gripper_ar_height}">
+      <xacro:inertial_box mass = "${1.587573295/3}" x = "${gripper_arm_length}" y = "${gripper_arm_width}" z = "${gripper_arm_height}">
         <origin xyz = "0 0 0" rpy = "0 0 0"/>
       </xacro:inertial_box>
@@ -72,5 +72,5 @@
     <!-- Right -->
     <link name="${prefix}_gripper_right_arm_link">
-      <xacro:inertial_box mass = "${1.587573295/3}" x = "${gripper_ar_length}" y = "${gripper_ar_width}" z = "${gripper_ar_height}">
+      <xacro:inertial_box mass = "${1.587573295/3}" x = "${gripper_arm_length}" y = "${gripper_arm_width}" z = "${gripper_arm_height}">
         <origin xyz = "0 0 0" rpy = "0 0 0"/>
       </xacro:inertial_box>

File: src/edna_description/urdf/parts/zed_macro.urdf.xacro (robot description, xacro)
@@ -63,5 +63,5 @@
     <link name="${prefix}_camera_center">
       <xacro:inertial_box mass="0.23" x="0.17525" y="0.03025" z="0.0431">
-        <origin xyz="${screw_offset_x} 0 0 0 0" rpy="0 0 0" />
+        <origin xyz="${screw_offset_x} 0 0" rpy="0 0 0" />
       </xacro:inertial_box>
       <visual>
