Commit message: stuff

File: src/edna_description/urdf/parts/swerve_axle.xacro (robot description, xacro)
@@ -44,5 +44,6 @@
                 <origin xyz="0 0 0" rpy="${pi / 2} 0 0"/>
                 <geometry>
-                    <cylinder  length="${wheel_length}" radius="${wheel_radius}"/>
+                    <cylinder length="${wheel_length}" radius="${wheel_radius}"/>
+                    <!-- <mesh filename="package://edna_description/meshes/SwerveWheel.stl" scale="0.001 0.001 0.001" /> -->
                 </geometry>
             </collision>
