Commit message: chonky robot

File: src/edna_description/urdf/parts/square_chassis.xacro (robot description, xacro)
@@ -5,5 +5,6 @@
   <xacro:property name="chassis_width" value=".7366" />
   <xacro:property name="chassis_height" value="0.05588" />
-  <xacro:property name="chassis_weight" value="38.55535145" />
+  <xacro:property name="chassis_weight" value="85" />
+  <!-- 38.55535145 -->
   <xacro:macro name="square_chassis" params="prefix parent *origin">
     <link name="${prefix}_chassis_link">

Commit message: bumper

File: src/edna_description/urdf/parts/square_chassis.xacro (robot description, xacro)
@@ -6,4 +6,8 @@
   <xacro:property name="chassis_height" value="0.05588" />
   <xacro:property name="chassis_weight" value="85" />
+  <xacro:property name="bumper_length" value="0.8128" />
+  <xacro:property name="bumper_width" value="0.8128" />
+  <xacro:property name="bumper_height" value="0.127" />
+  <xacro:property name="bumper_weight" value="6.80388555" />
   <!-- 38.55535145 -->
   <xacro:macro name="square_chassis" params="prefix parent *origin">
@@ -26,4 +30,22 @@
       </collision>
     </link>
+    <link name="${prefix}_bumper_link">
+      <xacro:inertial_box mass="${bumper_weight}" x="${bumper_length}" y="${bumper_width}" z="${bumper_height}">
+        <origin xyz="0 0 ${bumper_height/2}" rpy="0 0 0" />
+      </xacro:inertial_box>
+      <visual>
+        <origin xyz="0 0 ${bumper_height}" rpy="0 0 0" />
+        <geometry>
+          <mesh filename="package://edna_description/meshes/Bumper.stl" scale="0.001 0.001 0.001" />
+        </geometry>
+        <material name="blue"/>
+      </visual>
+      <collision>
+        <origin xyz="0 0 ${bumper_height/2}" rpy="0 0 0" />
+        <geometry>
+          <box size="${bumper_length} ${bumper_width} ${bumper_height} " />
+        </geometry>
+      </collision>
+    </link>
     <joint name="${prefix}_chassis_joint" type="fixed">
       <parent link="${parent}" />
@@ -31,4 +53,9 @@
       <xacro:insert_block name="origin" />
     </joint>
+    <joint name="${prefix}_bumper_joint" type="fixed">
+      <parent link="${parent}" />
+      <child link="${prefix}_bumper_link" />
+      <xacro:insert_block name="origin" />
+    </joint>
   </xacro:macro>
 </robot>

File: src/edna_description/urdf/util/materials.xacro (robot description, xacro)
@@ -6,4 +6,7 @@
   <material name="blue">
     <color rgba="${35/255} ${110/255} ${150/255} 1.0" />
+  </material>
+  <material name="dark-blue">
+    <color rgba="${0/255} ${0/255} ${139/255} 1.0" />
   </material>
   <material name="green">

Commit message: more bumpers

File: src/edna_description/urdf/parts/square_chassis.xacro (robot description, xacro)
@@ -39,5 +39,5 @@
           <mesh filename="package://edna_description/meshes/Bumper.stl" scale="0.001 0.001 0.001" />
         </geometry>
-        <material name="blue"/>
+        <material name="dark-blue"/>
       </visual>
       <collision>

Commit message: 1 inch

File: src/edna_description/urdf/parts/square_chassis.xacro (robot description, xacro)
@@ -32,8 +32,8 @@
     <link name="${prefix}_bumper_link">
       <xacro:inertial_box mass="${bumper_weight}" x="${bumper_length}" y="${bumper_width}" z="${bumper_height}">
-        <origin xyz="0 0 ${bumper_height/2}" rpy="0 0 0" />
+        <origin xyz="0 0 ${bumper_height/2 + 0.0254}" rpy="0 0 0" />
       </xacro:inertial_box>
       <visual>
-        <origin xyz="0 0 ${bumper_height}" rpy="0 0 0" />
+        <origin xyz="0 0 ${bumper_height + 0.0254}" rpy="0 0 0" />
         <geometry>
           <mesh filename="package://edna_description/meshes/Bumper.stl" scale="0.001 0.001 0.001" />
@@ -42,5 +42,5 @@
       </visual>
       <collision>
-        <origin xyz="0 0 ${bumper_height/2}" rpy="0 0 0" />
+        <origin xyz="0 0 ${bumper_height/2 + 0.0254}" rpy="0 0 0" />
         <geometry>
           <box size="${bumper_length} ${bumper_width} ${bumper_height} " />

Commit message: down

File: src/edna_description/urdf/parts/square_chassis.xacro (robot description, xacro)
@@ -32,8 +32,8 @@
     <link name="${prefix}_bumper_link">
       <xacro:inertial_box mass="${bumper_weight}" x="${bumper_length}" y="${bumper_width}" z="${bumper_height}">
-        <origin xyz="0 0 ${bumper_height/2 + 0.0254}" rpy="0 0 0" />
+        <origin xyz="0 0 ${bumper_height/2 + 0.0127}" rpy="0 0 0" />
       </xacro:inertial_box>
       <visual>
-        <origin xyz="0 0 ${bumper_height + 0.0254}" rpy="0 0 0" />
+        <origin xyz="0 0 ${bumper_height + 0.0127}" rpy="0 0 0" />
         <geometry>
           <mesh filename="package://edna_description/meshes/Bumper.stl" scale="0.001 0.001 0.001" />
@@ -42,5 +42,5 @@
       </visual>
       <collision>
-        <origin xyz="0 0 ${bumper_height/2 + 0.0254}" rpy="0 0 0" />
+        <origin xyz="0 0 ${bumper_height/2 + 0.0127}" rpy="0 0 0" />
         <geometry>
           <box size="${bumper_length} ${bumper_width} ${bumper_height} " />
