Commit message: poof

File: src/edna_description/urdf/parts/zed_macro.urdf.xacro (robot description, xacro)
@@ -62,7 +62,4 @@
     <!-- Camera Center -->
     <link name="${prefix}_camera_center">
-      <xacro:inertial_box mass="0.23" x="0.17525" y="0.03025" z="0.0431">
-        <origin xyz="${screw_offset_x} 0 0" rpy="0 0 0" />
-      </xacro:inertial_box>
       <visual>
         <origin xyz="${screw_offset_x} 0 0" rpy="0 0 0"/>
@@ -88,17 +85,11 @@
       <parent link="${prefix}_camera_center"/>
       <child link="${prefix}_left_camera_frame"/>
-      <origin xyz="0 ${baseline/2} 0" rpy="0 0 0" />
+      <origin xyz="0 ${baseline/2} 0" rpy="-${M_PI/2} 0 -${M_PI/2}" />
     </joint>
     <link name="${prefix}_left_camera_optical_frame"/>
     <joint name="${prefix}_left_camera_optical_joint" type="fixed">
-      <origin xyz="${optical_offset_x} 0 0" rpy="-${M_PI/2} 0.0 -${M_PI/2}"/>
+      <origin xyz="0 0 ${optical_offset_x}" rpy="${M_PI} 0 0"/>
       <parent link="${prefix}_left_camera_frame"/>
       <child link="${prefix}_left_camera_optical_frame"/>
-    </joint>
-    <link name="${prefix}_left_camera_isaac_frame"/>
-    <joint name="${prefix}_left_camera_isaac_joint" type="fixed">
-      <origin xyz="0 0 0" rpy="${M_PI/2} 0.0 -${M_PI/2}"/>
-      <parent link="${prefix}_left_camera_frame"/>
-      <child link="${prefix}_left_camera_isaac_frame"/>
     </joint>
     <!-- Right Camera -->
@@ -107,24 +98,39 @@
       <parent link="${prefix}_camera_center"/>
       <child link="${prefix}_right_camera_frame"/>
-      <origin xyz="0 -${baseline/2} 0" rpy="0 0 0" />
+      <origin xyz="0 -${baseline/2} 0" rpy="-${M_PI/2} 0 -${M_PI/2}" />
     </joint>
     <link name="${prefix}_right_camera_optical_frame"/>
     <joint name="${prefix}_right_camera_optical_joint" type="fixed">
-      <origin xyz="${optical_offset_x} 0 0" rpy="-${M_PI/2} 0.0 -${M_PI/2}"/>
+      <origin xyz="0 0 ${optical_offset_x}" rpy="${M_PI} 0 0"/>
       <parent link="${prefix}_right_camera_frame"/>
       <child link="${prefix}_right_camera_optical_frame"/>
     </joint>
-    <link name="${prefix}_right_camera_isaac_frame"/>
-    <joint name="${prefix}_right_camera_isaac_joint" type="fixed">
-      <origin xyz="0 0 0" rpy="${M_PI/2} 0.0 -${M_PI/2}"/>
-      <parent link="${prefix}_right_camera_frame"/>
-      <child link="${prefix}_right_camera_isaac_frame"/>
-    </joint>
-    <link name="${prefix}_imu_link" />
-    <joint name="${prefix}_imu_joint" type="fixed">
-      <parent link="${prefix}_left_camera_frame"/>
-      <child link="${prefix}_imu_link"/>
-      <origin xyz="0 0 0" rpy="0 0 0" />
-    </joint>
+    <!-- ZED2 Sensors -->
+    <xacro:if value="${model == 'zed2'}">
+      <link name="${prefix}_mag_link" />
+      <joint name="${prefix}_mag_joint" type="fixed">
+        <parent link="${prefix}_camera_center"/>
+        <child link="${prefix}_mag_link"/>
+        <origin xyz="0 0 0" rpy="0 0 0" />
+      </joint>
+      <link name="${prefix}_baro_link" />
+      <joint name="${prefix}_baro_joint" type="fixed">
+        <parent link="${prefix}_camera_center"/>
+        <child link="${prefix}_baro_link"/>
+        <origin xyz="0 0 0" rpy="0 0 0" />
+      </joint>
+      <link name="${prefix}_temp_left_link" />
+      <joint name="${prefix}_temp_left_joint" type="fixed">
+        <parent link="${prefix}_left_camera_frame"/>
+        <child link="${prefix}_temp_left_link"/>
+        <origin xyz="0 0 0" rpy="0 0 0" />
+      </joint>
+      <link name="${prefix}_temp_right_link" />
+      <joint name="${prefix}_temp_right_joint" type="fixed">
+        <parent link="${prefix}_right_camera_frame"/>
+        <child link="${prefix}_temp_right_link"/>
+        <origin xyz="0 0 0" rpy="0 0 0" />
+      </joint>
+    </xacro:if>
   </xacro:macro>
 </robot>

Commit message: imu

File: src/edna_description/urdf/parts/zed_macro.urdf.xacro (robot description, xacro)
@@ -85,5 +85,5 @@
       <parent link="${prefix}_camera_center"/>
       <child link="${prefix}_left_camera_frame"/>
-      <origin xyz="0 ${baseline/2} 0" rpy="-${M_PI/2} 0 -${M_PI/2}" />
+      <origin xyz="0 ${baseline/2} 0" rpy="-${M_PI/2} ${M_PI} ${M_PI/2}" />
     </joint>
     <link name="${prefix}_left_camera_optical_frame"/>
@@ -98,5 +98,5 @@
       <parent link="${prefix}_camera_center"/>
       <child link="${prefix}_right_camera_frame"/>
-      <origin xyz="0 -${baseline/2} 0" rpy="-${M_PI/2} 0 -${M_PI/2}" />
+      <origin xyz="0 -${baseline/2} 0" rpy="-${M_PI/2} ${M_PI} ${M_PI/2}" />
     </joint>
     <link name="${prefix}_right_camera_optical_frame"/>

Commit message: WORKING RTAB MAP

File: src/edna_description/urdf/parts/zed_macro.urdf.xacro (robot description, xacro)
@@ -85,5 +85,5 @@
       <parent link="${prefix}_camera_center"/>
       <child link="${prefix}_left_camera_frame"/>
-      <origin xyz="0 ${baseline/2} 0" rpy="-${M_PI/2} ${M_PI} ${M_PI/2}" />
+      <origin xyz="0 ${baseline/2} 0" rpy="-${M_PI/2} 0 -${M_PI/2}" />
     </joint>
     <link name="${prefix}_left_camera_optical_frame"/>
@@ -98,5 +98,5 @@
       <parent link="${prefix}_camera_center"/>
       <child link="${prefix}_right_camera_frame"/>
-      <origin xyz="0 -${baseline/2} 0" rpy="-${M_PI/2} ${M_PI} ${M_PI/2}" />
+      <origin xyz="0 -${baseline/2} 0" rpy="-${M_PI/2} 0 -${M_PI/2}" />
     </joint>
     <link name="${prefix}_right_camera_optical_frame"/>

Commit message: gym/urdf changes

File: src/edna_description/urdf/parts/zed_macro.urdf.xacro (robot description, xacro)
@@ -52,4 +52,5 @@
       <xacro:property name="screw_offset_x" value="-0.01" />
       <xacro:property name="optical_offset_x" value="-0.01" />
+      <xacro:property name="weight" value="0.166" />
     </xacro:if>
     <!-- Camera mounting point (the threaded screw hole in the bottom) -->
@@ -81,5 +82,9 @@
     </joint>
     <!-- Left Camera -->
-    <link name="${prefix}_left_camera_frame" />
+    <link name="${prefix}_left_camera_frame">
+      <xacro:inertial_box mass="${weight/4}" x="0.0" y="0.0" z="0.0">
+        <origin xyz="0 ${baseline/2} 0" rpy="0 0 0" />
+      </xacro:inertial_box>
+    </link>
     <joint name="${prefix}_left_camera_joint" type="fixed">
       <parent link="${prefix}_camera_center"/>
@@ -87,5 +92,9 @@
       <origin xyz="0 ${baseline/2} 0" rpy="-${M_PI/2} 0 -${M_PI/2}" />
     </joint>
-    <link name="${prefix}_left_camera_optical_frame"/>
+    <link name="${prefix}_left_camera_optical_frame">
+      <xacro:inertial_box mass="${weight/4}" x="0.0" y="0.0" z="0.0">
+        <origin xyz="0 ${baseline/2} 0" rpy="0 0 0" />
+      </xacro:inertial_box>
+    </link>
     <joint name="${prefix}_left_camera_optical_joint" type="fixed">
       <origin xyz="0 0 ${optical_offset_x}" rpy="${M_PI} 0 0"/>
@@ -94,5 +103,9 @@
     </joint>
     <!-- Right Camera -->
-    <link name="${prefix}_right_camera_frame" />
+    <link name="${prefix}_right_camera_frame">
+      <xacro:inertial_box mass="${weight/4}" x="0.0" y="0.0" z="0.0">
+        <origin xyz="0 ${baseline/2} 0" rpy="0 0 0" />
+      </xacro:inertial_box>
+    </link>
     <joint name="${prefix}_right_camera_joint" type="fixed">
       <parent link="${prefix}_camera_center"/>
@@ -100,5 +113,9 @@
       <origin xyz="0 -${baseline/2} 0" rpy="-${M_PI/2} 0 -${M_PI/2}" />
     </joint>
-    <link name="${prefix}_right_camera_optical_frame"/>
+    <link name="${prefix}_right_camera_optical_frame">
+      <xacro:inertial_box mass="${weight/4}" x="0.0" y="0.0" z="0.0">
+        <origin xyz="0 ${baseline/2} 0" rpy="0 0 0" />
+      </xacro:inertial_box>
+    </link>
     <joint name="${prefix}_right_camera_optical_joint" type="fixed">
       <origin xyz="0 0 ${optical_offset_x}" rpy="${M_PI} 0 0"/>
